Commit message: Added simulation worlds, and camera and depth camera functionality

File: robots/g1_description/xacro/gazebo.xacro (robot description, xacro)
@@ -34,3 +34,66 @@
         <mu2>0.2</mu2>
     </gazebo>
+    <!-- Elimina la configuración anterior de la cámara y añade esta -->
+    <!-- Gazebo sensor definitions for simulating the RealSense D435i -->
+    <gazebo reference="head_link">
+      <sensor type="camera" name="realsense_rgb_camera">
+        <update_rate>30.0</update_rate>
+        <camera>
+          <horizontal_fov>1.3962634</horizontal_fov>
+          <image>
+            <width>640</width>
+            <height>480</height>
+            <format>R8G8B8</format>
+          </image>
+          <clip>
+            <near>0.1</near>
+            <far>100.0</far>
+          </clip>
+        </camera>
+        <plugin name="realsense_rgb_plugin" filename="libgazebo_ros_camera.so">
+          <alwaysOn>true</alwaysOn>
+          <updateRate>30.0</updateRate>
+          <cameraName>realsense</cameraName>
+          <imageTopicName>rgb/image_raw</imageTopicName>
+          <cameraInfoTopicName>rgb/camera_info</cameraInfoTopicName>
+          <frameName>realsense_rgb_frame</frameName>
+          <hackBaseline>0.07</hackBaseline>
+          <distortionK1>0.0</distortionK1>
+          <distortionK2>0.0</distortionK2>
+          <distortionK3>0.0</distortionK3>
+          <distortionT1>0.0</distortionT1>
+          <distortionT2>0.0</distortionT2>
+        </plugin>
+      </sensor>
+      <sensor type="depth" name="realsense_depth_camera">
+        <update_rate>30.0</update_rate>
+        <camera>
+          <horizontal_fov>1.3962634</horizontal_fov>
+          <image>
+            <width>640</width>
+            <height>480</height>
+            <format>R8G8B8</format>
+          </image>
+          <clip>
+            <near>0.1</near>
+            <far>10.0</far>
+          </clip>
+        </camera>
+        <plugin name="realsense_depth_plugin" filename="libgazebo_ros_depth_camera.so">
+          <alwaysOn>true</alwaysOn>
+          <updateRate>30.0</updateRate>
+          <cameraName>realsense</cameraName>
+          <imageTopicName>depth/image_raw</imageTopicName>
+          <cameraInfoTopicName>depth/camera_info</cameraInfoTopicName>
+          <pointCloudTopicName>depth/points</pointCloudTopicName>
+          <frameName>realsense_depth_frame</frameName>
+          <hackBaseline>0.07</hackBaseline>
+          <distortionK1>0.0</distortionK1>
+          <distortionK2>0.0</distortionK2>
+          <distortionK3>0.0</distortionK3>
+          <distortionT1>0.0</distortionT1>
+          <distortionT2>0.0</distortionT2>
+        </plugin>
+      </sensor>
+    </gazebo>
 </robot>

File: robots/g1_description/xacro/robot.xacro (robot description, xacro)
@@ -241,4 +241,42 @@
     <child link="head_link"/>
   </joint>
+  <!-- Frames adicionales para la RealSense -->
+  <link name="realsense_rgb_frame"/>
+  <joint name="realsense_rgb_joint" type="fixed">
+    <origin xyz="0.06 0 0.48" rpy="0 0 0"/>
+    <parent link="head_link"/>
+    <child link="realsense_rgb_frame"/>
+  </joint>
+  <link name="realsense_depth_frame"/>
+  <joint name="realsense_depth_joint" type="fixed">
+    <origin xyz="0.06 0 0.48" rpy="0 0 0"/>
+    <parent link="head_link"/>
+    <child link="realsense_depth_frame"/>
+  </joint>
+  <!-- Camera link -->
+  <link name="camera_link">
+    <visual>
+      <origin xyz="0 0 0" rpy="0 0 0"/>
+      <geometry>
+        <box size="0.01 0.01 0.01"/>
+      </geometry>
+      <material name="">
+        <color rgba="0 0 0 1"/>
+      </material>
+    </visual>
+  </link>
+  <!-- Camera joint - posicionada en la parte frontal de la cabeza -->
+  <joint name="camera_joint" type="fixed">
+    <origin xyz="0.06 0 0.48" rpy="0 0 0"/>
+    <parent link="head_link"/>
+    <child link="camera_link"/>
+  </joint>
+  <!-- Camera optical frame -->
+  <link name="camera_optical_frame"/>
+  <joint name="camera_optical_joint" type="fixed">
+    <origin xyz="0 0 0" rpy="-1.57079632679 0 -1.57079632679"/>
+    <parent link="camera_link"/>
+    <child link="camera_optical_frame"/>
+  </joint>
   <!-- IMU -->
   <link name="imu_link"></link>
