Commit message: Added livox lidar functionality

File: robots/g1_description/xacro/gazebo.xacro (robot description, xacro)
@@ -1,99 +1,142 @@
 <?xml version="1.0"?>
 <robot>
-    <!-- ros_control plugin -->
-    <gazebo>
-        <plugin name="gazebo_ros_control" filename="libgazebo_ros_control.so">
-            <robotNamespace>/g1_gazebo</robotNamespace>
-            <robotSimType>gazebo_ros_control/DefaultRobotHWSim</robotSimType>
-        </plugin>
-    </gazebo>
-    <gazebo reference="imu_link">
-        <gravity>true</gravity>
-        <sensor name="imu_sensor" type="imu">
-            <always_on>true</always_on>
-            <update_rate>1000</update_rate>
-            <visualize>true</visualize>
-            <topic>__default_topic__</topic>
-            <plugin filename="libgazebo_ros_imu_sensor.so" name="imu_plugin">
-                <topicName>trunk_imu</topicName>
-                <bodyName>imu_link</bodyName>
-                <updateRateHZ>1000.0</updateRateHZ>
-                <gaussianNoise>0.0</gaussianNoise>
-                <xyzOffset>0 0 0</xyzOffset>
-                <rpyOffset>0 0 0</rpyOffset>
-                <frameName>imu_link</frameName>
-            </plugin>
-            <pose>0 0 0 0 0 0</pose>
-        </sensor>
-    </gazebo>
-    <gazebo reference="base">
-        <turnGravityOff>false</turnGravityOff>
-    </gazebo>
-    <gazebo reference="imu_link">
-        <mu1>0.2</mu1>
-        <mu2>0.2</mu2>
-    </gazebo>
-    <!-- Elimina la configuración anterior de la cámara y añade esta -->
-    <!-- Gazebo sensor definitions for simulating the RealSense D435i -->
-    <gazebo reference="head_link">
-      <sensor type="camera" name="realsense_rgb_camera">
-        <update_rate>30.0</update_rate>
-        <camera>
-          <horizontal_fov>1.3962634</horizontal_fov>
-          <image>
-            <width>640</width>
-            <height>480</height>
-            <format>R8G8B8</format>
-          </image>
-          <clip>
-            <near>0.1</near>
-            <far>100.0</far>
-          </clip>
-        </camera>
-        <plugin name="realsense_rgb_plugin" filename="libgazebo_ros_camera.so">
-          <alwaysOn>true</alwaysOn>
-          <updateRate>30.0</updateRate>
-          <cameraName>realsense</cameraName>
-          <imageTopicName>rgb/image_raw</imageTopicName>
-          <cameraInfoTopicName>rgb/camera_info</cameraInfoTopicName>
-          <frameName>realsense_rgb_frame</frameName>
-          <hackBaseline>0.07</hackBaseline>
-          <distortionK1>0.0</distortionK1>
-          <distortionK2>0.0</distortionK2>
-          <distortionK3>0.0</distortionK3>
-          <distortionT1>0.0</distortionT1>
-          <distortionT2>0.0</distortionT2>
-        </plugin>
-      </sensor>
-      <sensor type="depth" name="realsense_depth_camera">
-        <update_rate>30.0</update_rate>
-        <camera>
-          <horizontal_fov>1.3962634</horizontal_fov>
-          <image>
-            <width>640</width>
-            <height>480</height>
-            <format>R8G8B8</format>
-          </image>
-          <clip>
-            <near>0.1</near>
-            <far>10.0</far>
-          </clip>
-        </camera>
-        <plugin name="realsense_depth_plugin" filename="libgazebo_ros_depth_camera.so">
-          <alwaysOn>true</alwaysOn>
-          <updateRate>30.0</updateRate>
-          <cameraName>realsense</cameraName>
-          <imageTopicName>depth/image_raw</imageTopicName>
-          <cameraInfoTopicName>depth/camera_info</cameraInfoTopicName>
-          <pointCloudTopicName>depth/points</pointCloudTopicName>
-          <frameName>realsense_depth_frame</frameName>
-          <hackBaseline>0.07</hackBaseline>
-          <distortionK1>0.0</distortionK1>
-          <distortionK2>0.0</distortionK2>
-          <distortionK3>0.0</distortionK3>
-          <distortionT1>0.0</distortionT1>
-          <distortionT2>0.0</distortionT2>
-        </plugin>
-      </sensor>
-    </gazebo>
+  <!-- ros_control plugin -->
+  <gazebo>
+    <plugin name="gazebo_ros_control" filename="libgazebo_ros_control.so">
+      <robotNamespace>/g1_gazebo</robotNamespace>
+      <robotSimType>gazebo_ros_control/DefaultRobotHWSim</robotSimType>
+    </plugin>
+  </gazebo>
+  <gazebo reference="imu_link">
+    <gravity>true</gravity>
+    <sensor name="imu_sensor" type="imu">
+      <always_on>true</always_on>
+      <update_rate>1000</update_rate>
+      <visualize>true</visualize>
+      <topic>__default_topic__</topic>
+      <plugin filename="libgazebo_ros_imu_sensor.so" name="imu_plugin">
+        <topicName>trunk_imu</topicName>
+        <bodyName>imu_link</bodyName>
+        <updateRateHZ>1000.0</updateRateHZ>
+        <gaussianNoise>0.0</gaussianNoise>
+        <xyzOffset>0 0 0</xyzOffset>
+        <rpyOffset>0 0 0</rpyOffset>
+        <frameName>imu_link</frameName>
+      </plugin>
+      <pose>0 0 0 0 0 0</pose>
+    </sensor>
+  </gazebo>
+  <gazebo reference="base">
+    <turnGravityOff>false</turnGravityOff>
+  </gazebo>
+  <gazebo reference="imu_link">
+    <mu1>0.2</mu1>
+    <mu2>0.2</mu2>
+  </gazebo>
+  <!-- Elimina la configuración anterior de la cámara y añade esta -->
+  <!-- Gazebo sensor definitions for simulating the RealSense D435i -->
+  <gazebo reference="head_link">
+    <sensor type="camera" name="realsense_rgb_camera">
+      <update_rate>30.0</update_rate>
+      <camera>
+        <horizontal_fov>1.3962634</horizontal_fov>
+        <image>
+          <width>640</width>
+          <height>480</height>
+          <format>R8G8B8</format>
+        </image>
+        <clip>
+          <near>0.1</near>
+          <far>100.0</far>
+        </clip>
+      </camera>
+      <plugin name="realsense_rgb_plugin" filename="libgazebo_ros_camera.so">
+        <alwaysOn>true</alwaysOn>
+        <updateRate>30.0</updateRate>
+        <cameraName>realsense</cameraName>
+        <imageTopicName>rgb/image_raw</imageTopicName>
+        <cameraInfoTopicName>rgb/camera_info</cameraInfoTopicName>
+        <frameName>realsense_rgb_frame</frameName>
+        <hackBaseline>0.07</hackBaseline>
+        <distortionK1>0.0</distortionK1>
+        <distortionK2>0.0</distortionK2>
+        <distortionK3>0.0</distortionK3>
+        <distortionT1>0.0</distortionT1>
+        <distortionT2>0.0</distortionT2>
+      </plugin>
+    </sensor>
+    <sensor type="depth" name="realsense_depth_camera">
+      <update_rate>30.0</update_rate>
+      <camera>
+        <horizontal_fov>1.3962634</horizontal_fov>
+        <image>
+          <width>640</width>
+          <height>480</height>
+          <format>R8G8B8</format>
+        </image>
+        <clip>
+          <near>0.1</near>
+          <far>10.0</far>
+        </clip>
+      </camera>
+      <plugin name="realsense_depth_plugin" filename="libgazebo_ros_depth_camera.so">
+        <alwaysOn>true</alwaysOn>
+        <updateRate>30.0</updateRate>
+        <cameraName>realsense</cameraName>
+        <imageTopicName>depth/image_raw</imageTopicName>
+        <cameraInfoTopicName>depth/camera_info</cameraInfoTopicName>
+        <pointCloudTopicName>depth/points</pointCloudTopicName>
+        <frameName>realsense_depth_frame</frameName>
+        <hackBaseline>0.07</hackBaseline>
+        <distortionK1>0.0</distortionK1>
+        <distortionK2>0.0</distortionK2>
+        <distortionK3>0.0</distortionK3>
+        <distortionT1>0.0</distortionT1>
+        <distortionT2>0.0</distortionT2>
+      </plugin>
+    </sensor>
+  </gazebo>
+  <gazebo reference="head_link">
+    <sensor type="ray" name="livox_lidar">
+      <pose>0.06 0 0.5 0 0 0</pose>
+      <visualize>false</visualize>
+      <always_on>true</always_on>
+      <update_rate>10</update_rate>
+      <plugin name="gazebo_ros_laser_controller" filename="liblivox_laser_simulation.so">
+        <ray>
+          <scan>
+            <horizontal>
+              <samples>100</samples>
+              <resolution>1</resolution>
+              <min_angle>-3.1415926535897931</min_angle>
+              <max_angle>3.1415926535897931</max_angle>
+            </horizontal>
+            <vertical>
+              <samples>50</samples>
+              <resolution>1</resolution>
+              <min_angle>-3.1415926535897931</min_angle>
+              <max_angle>3.1415926535897931</max_angle>
+            </vertical>
+          </scan>
+          <range>
+            <min>0.1</min>
+            <max>40</max>
+            <resolution>1</resolution>
+          </range>
+          <noise>
+            <type>gaussian</type>
+            <mean>0.0</mean>
+            <stddev>0.0</stddev>
+          </noise>
+        </ray>
+        <visualize>true</visualize>
+        <samples>20000</samples>
+        <downsample>1</downsample>
+        <csv_file_name>mid360-real-centr.csv</csv_file_name>
+        <publish_pointcloud_type>2</publish_pointcloud_type>
+        <ros_topic>/livox/lidar</ros_topic>
+        <frameName>livox_lidar_frame</frameName>
+      </plugin>
+    </sensor>
+  </gazebo>
 </robot>

File: robots/g1_description/xacro/robot.xacro (robot description, xacro)
@@ -1,266 +1,270 @@
 <?xml version="1.0"?>
 <robot name="g1_description" xmlns:xacro="http://www.ros.org/wiki/xacro">
-  <xacro:arg name="DEBUG" default="false"/>
-  <xacro:include filename="$(find g1_description)/xacro/gazebo.xacro"/>
-  <xacro:include filename="$(find g1_description)/xacro/const.xacro"/>
-  <xacro:include filename="$(find g1_description)/xacro/leg.xacro"/>
-  <xacro:include filename="$(find g1_description)/xacro/arm.xacro"/>
+  <xacro:arg name="DEBUG" default="false" />
+  <xacro:include filename="$(find g1_description)/xacro/gazebo.xacro" />
+  <xacro:include filename="$(find g1_description)/xacro/const.xacro" />
+  <xacro:include filename="$(find g1_description)/xacro/leg.xacro" />
+  <xacro:include filename="$(find g1_description)/xacro/arm.xacro" />
   <!-- Rotor related joint and link is only for demonstrate location. -->
-  <!-- Actually, the rotor will rotate and the joint is not fixed. Reduction ratio should be considered. -->
+  <!-- Actually, the rotor will rotate and the joint is not fixed. Reduction ratio should be
+  considered. -->
   <!-- Debug mode will hung up the robot, use "true" or "false" to switch it. -->
   <xacro:if value="$(arg DEBUG)">
-      <link name="world"/>
-      <joint name="base_static_joint" type="fixed">
-          <origin rpy="0 0 0" xyz="0 0 0.5"/>
-          <parent link="world"/>
-          <child link="pelvis"/>
-      </joint>
+    <link name="world" />
+    <joint name="base_static_joint" type="fixed">
+      <origin rpy="0 0 0" xyz="0 0 0.5" />
+      <parent link="world" />
+      <child link="pelvis" />
+    </joint>
   </xacro:if>
- <!-- Torso -->
+  <!-- Torso -->
   <link name="torso_link">
     <inertial>
-      <origin xyz="${torso_link_com_x} ${torso_link_com_y} ${torso_link_com_z}" rpy="0 0 0"/>
-      <mass value="${torso_link_mass}"/>
+      <origin xyz="${torso_link_com_x} ${torso_link_com_y} ${torso_link_com_z}" rpy="0 0 0" />
+      <mass value="${torso_link_mass}" />
       <inertia
         ixx="${torso_link_ixx}" ixy="${torso_link_ixy}" ixz="${torso_link_ixz}"
         iyy="${torso_link_iyy}" iyz="${torso_link_iyz}"
-        izz="${torso_link_izz}"/>
+        izz="${torso_link_izz}" />
     </inertial>
     <visual>
-      <origin xyz="0 0 0" rpy="0 0 0"/>
-      <geometry>
-        <mesh filename="package://g1_description/meshes/torso_link.STL"/>
-      </geometry>
-      <material name="">
-        <color rgba="0.7 0.7 0.7 1"/>
-      </material>
-    </visual>
-    <collision>
-        <origin xyz="0.055 0.055 -0.020" rpy="0 0 0"/>
-        <geometry>
-        <sphere radius="0.01"/>
-        </geometry>
-    </collision>
-    <collision>
-        <origin xyz="0.055 -0.055 -0.020" rpy="0 0 0"/>
-        <geometry>
-        <sphere radius="0.01"/>
-        </geometry>
-    </collision>
-    <collision>
-        <origin xyz="-0.055 0.055 -0.020" rpy="0 0 0"/>
-        <geometry>
-        <sphere radius="0.01"/>
-        </geometry>
-    </collision>
-    <collision>
-        <origin xyz="-0.055 -0.055 -0.020" rpy="0 0 0"/>
-        <geometry>
-        <sphere radius="0.01"/>
-        </geometry>
-    </collision>
-    <collision>
-        <origin xyz="0.063 0.088 0.065" rpy="0 0 0"/>
-        <geometry>
-        <sphere radius="0.01"/>
-        </geometry>
-    </collision>
-    <collision>
-        <origin xyz="0.063 -0.088 0.065" rpy="0 0 0"/>
-        <geometry>
-        <sphere radius="0.01"/>
-        </geometry>
-    </collision>
-    <collision>
-        <origin xyz="-0.063 0.088 0.065" rpy="0 0 0"/>
-        <geometry>
-        <sphere radius="0.01"/>
-        </geometry>
-    </collision>
-    <collision>
-        <origin xyz="-0.063 -0.088 0.065" rpy="0 0 0"/>
-        <geometry>
-        <sphere radius="0.01"/>
-        </geometry>
-    </collision>
-    <collision>
-        <origin xyz="0.063 0.088 0.30" rpy="0 0 0"/>
-        <geometry>
-        <sphere radius="0.01"/>
-        </geometry>
-    </collision>
-    <collision>
-        <origin xyz="0.063 -0.088 0.30" rpy="0 0 0"/>
-        <geometry>
-        <sphere radius="0.01"/>
-        </geometry>
-    </collision>
-    <collision>
-        <origin xyz="-0.066 0.088 0.30" rpy="0 0 0"/>
-        <geometry>
-        <sphere radius="0.01"/>
-        </geometry>
-    </collision>
-    <collision>
-        <origin xyz="-0.066 -0.088 0.30" rpy="0 0 0"/>
-        <geometry>
-        <sphere radius="0.01"/>
-        </geometry>
+      <origin xyz="0 0 0" rpy="0 0 0" />
+      <geometry>
+        <mesh filename="package://g1_description/meshes/torso_link.STL" />
+      </geometry>
+      <material name="">
+        <color rgba="0.7 0.7 0.7 1" />
+      </material>
+    </visual>
+    <collision>
+      <origin xyz="0.055 0.055 -0.020" rpy="0 0 0" />
+      <geometry>
+        <sphere radius="0.01" />
+      </geometry>
+    </collision>
+    <collision>
+      <origin xyz="0.055 -0.055 -0.020" rpy="0 0 0" />
+      <geometry>
+        <sphere radius="0.01" />
+      </geometry>
+    </collision>
+    <collision>
+      <origin xyz="-0.055 0.055 -0.020" rpy="0 0 0" />
+      <geometry>
+        <sphere radius="0.01" />
+      </geometry>
+    </collision>
+    <collision>
+      <origin xyz="-0.055 -0.055 -0.020" rpy="0 0 0" />
+      <geometry>
+        <sphere radius="0.01" />
+      </geometry>
+    </collision>
+    <collision>
+      <origin xyz="0.063 0.088 0.065" rpy="0 0 0" />
+      <geometry>
+        <sphere radius="0.01" />
+      </geometry>
+    </collision>
+    <collision>
+      <origin xyz="0.063 -0.088 0.065" rpy="0 0 0" />
+      <geometry>
+        <sphere radius="0.01" />
+      </geometry>
+    </collision>
+    <collision>
+      <origin xyz="-0.063 0.088 0.065" rpy="0 0 0" />
+      <geometry>
+        <sphere radius="0.01" />
+      </geometry>
+    </collision>
+    <collision>
+      <origin xyz="-0.063 -0.088 0.065" rpy="0 0 0" />
+      <geometry>
+        <sphere radius="0.01" />
+      </geometry>
+    </collision>
+    <collision>
+      <origin xyz="0.063 0.088 0.30" rpy="0 0 0" />
+      <geometry>
+        <sphere radius="0.01" />
+      </geometry>
+    </collision>
+    <collision>
+      <origin xyz="0.063 -0.088 0.30" rpy="0 0 0" />
+      <geometry>
+        <sphere radius="0.01" />
+      </geometry>
+    </collision>
+    <collision>
+      <origin xyz="-0.066 0.088 0.30" rpy="0 0 0" />
+      <geometry>
+        <sphere radius="0.01" />
+      </geometry>
+    </collision>
+    <collision>
+      <origin xyz="-0.066 -0.088 0.30" rpy="0 0 0" />
+      <geometry>
+        <sphere radius="0.01" />
+      </geometry>
     </collision>
   </link>
   <joint name="torso_joint" type="revolute">
-    <origin xyz="${torso_joint_offset_x} ${torso_joint_offset_y} ${torso_joint_offset_z}" rpy="0 0 0"/>
-    <parent link="pelvis"/>
-    <child link="torso_link"/>
-    <axis xyz="0 0 1"/>
-    <limit lower="${torso_joint_position_min}" upper="${torso_joint_position_max}" effort="${torso_joint_torque_max}" velocity="${torso_joint_velocity_max}"/>
+    <origin xyz="${torso_joint_offset_x} ${torso_joint_offset_y} ${torso_joint_offset_z}"
+      rpy="0 0 0" />
+    <parent link="pelvis" />
+    <child link="torso_link" />
+    <axis xyz="0 0 1" />
+    <limit lower="${torso_joint_position_min}" upper="${torso_joint_position_max}"
+      effort="${torso_joint_torque_max}" velocity="${torso_joint_velocity_max}" />
   </joint>
   <link name="pelvis">
     <inertial>
-      <origin xyz="0 0 -0.07605" rpy="0 0 0"/>
-      <mass value="2.86"/>
-      <inertia ixx="0.0079143" ixy="0" ixz="1.6E-06" iyy="0.0069837" iyz="0" izz="0.0059404"/>
+      <origin xyz="0 0 -0.07605" rpy="0 0 0" />
+      <mass value="2.86" />
+      <inertia ixx="0.0079143" ixy="0" ixz="1.6E-06" iyy="0.0069837" iyz="0" izz="0.0059404" />
     </inertial>
     <visual>
-      <origin xyz="0 0 0" rpy="0 0 0"/>
-      <geometry>
-        <mesh filename="package://g1_description/meshes/pelvis.STL"/>
-      </geometry>
-      <material name="">
-        <color rgba="0.7 0.7 0.7 1"/>
-      </material>
-    </visual>
-    <collision>
-        <origin xyz="0.050 0.060 -0.060" rpy="0 0 0"/>
-        <geometry>
-        <sphere radius="0.01"/>
-        </geometry>
-    </collision>
-    <collision>
-        <origin xyz="0.050 -0.060 -0.060" rpy="0 0 0"/>
-        <geometry>
-        <sphere radius="0.01"/>
-        </geometry>
-    </collision>
-    <collision>
-        <origin xyz="-0.050 0.060 -0.060" rpy="0 0 0"/>
-        <geometry>
-        <sphere radius="0.01"/>
-        </geometry>
-    </collision>
-    <collision>
-        <origin xyz="-0.050 -0.060 -0.060" rpy="0 0 0"/>
-        <geometry>
-        <sphere radius="0.01"/>
-        </geometry>
-    </collision>
-    <collision>
-        <origin xyz="0.050 0.060 -0.135" rpy="0 0 0"/>
-        <geometry>
-        <sphere radius="0.01"/>
-        </geometry>
-    </collision>
-    <collision>
-        <origin xyz="0.050 -0.060 -0.135" rpy="0 0 0"/>
-        <geometry>
-        <sphere radius="0.01"/>
-        </geometry>
-    </collision>
-    <collision>
-        <origin xyz="-0.050 0.060 -0.135" rpy="0 0 0"/>
-        <geometry>
-        <sphere radius="0.01"/>
-        </geometry>
-    </collision>
-    <collision>
-        <origin xyz="-0.050 -0.060 -0.135" rpy="0 0 0"/>
-        <geometry>
-        <sphere radius="0.01"/>
-        </geometry>
+      <origin xyz="0 0 0" rpy="0 0 0" />
+      <geometry>
+        <mesh filename="package://g1_description/meshes/pelvis.STL" />
+      </geometry>
+      <material name="">
+        <color rgba="0.7 0.7 0.7 1" />
+      </material>
+    </visual>
+    <collision>
+      <origin xyz="0.050 0.060 -0.060" rpy="0 0 0" />
+      <geometry>
+        <sphere radius="0.01" />
+      </geometry>
+    </collision>
+    <collision>
+      <origin xyz="0.050 -0.060 -0.060" rpy="0 0 0" />
+      <geometry>
+        <sphere radius="0.01" />
+      </geometry>
+    </collision>
+    <collision>
+      <origin xyz="-0.050 0.060 -0.060" rpy="0 0 0" />
+      <geometry>
+        <sphere radius="0.01" />
+      </geometry>
+    </collision>
+    <collision>
+      <origin xyz="-0.050 -0.060 -0.060" rpy="0 0 0" />
+      <geometry>
+        <sphere radius="0.01" />
+      </geometry>
+    </collision>
+    <collision>
+      <origin xyz="0.050 0.060 -0.135" rpy="0 0 0" />
+      <geometry>
+        <sphere radius="0.01" />
+      </geometry>
+    </collision>
+    <collision>
+      <origin xyz="0.050 -0.060 -0.135" rpy="0 0 0" />
+      <geometry>
+        <sphere radius="0.01" />
+      </geometry>
+    </collision>
+    <collision>
+      <origin xyz="-0.050 0.060 -0.135" rpy="0 0 0" />
+      <geometry>
+        <sphere radius="0.01" />
+      </geometry>
+    </collision>
+    <collision>
+      <origin xyz="-0.050 -0.060 -0.135" rpy="0 0 0" />
+      <geometry>
+        <sphere radius="0.01" />
+      </geometry>
     </collision>
   </link>
   <link name="pelvis_contour_link">
     <visual>
-      <origin xyz="0 0 0" rpy="0 0 0"/>
-      <geometry>
-        <mesh filename="package://g1_description/meshes/pelvis_contour_link.STL"/>
-      </geometry>
-      <material name="">
-        <color rgba="0.2 0.2 0.2 1"/>
+      <origin xyz="0 0 0" rpy="0 0 0" />
+      <geometry>
+        <mesh filename="package://g1_description/meshes/pelvis_contour_link.STL" />
+      </geometry>
+      <material name="">
+        <color rgba="0.2 0.2 0.2 1" />
       </material>
     </visual>
   </link>
   <joint name="pelvis_contour_joint" type="fixed">
-    <parent link="pelvis"/>
-    <child link="pelvis_contour_link"/>
-  </joint>
- <!-- Head -->
+    <parent link="pelvis" />
+    <child link="pelvis_contour_link" />
+  </joint>
+  <!-- Head -->
   <link name="head_link">
     <inertial>
-      <origin xyz="0.00138066852 0.00028430950 0.42034187824" rpy="0 0 0"/>
-      <mass value="1.17976522"/>
-      <inertia ixx="0.00543236042361" ixy="0.00000140137425" ixz="0.00034554752228" iyy="0.00552885306699" iyz="0.00001501216392" izz="0.00165378108136"/>
+      <origin xyz="0.00138066852 0.00028430950 0.42034187824" rpy="0 0 0" />
+      <mass value="1.17976522" />
+      <inertia ixx="0.00543236042361" ixy="0.00000140137425" ixz="0.00034554752228"
+        iyy="0.00552885306699" iyz="0.00001501216392" izz="0.00165378108136" />
     </inertial>
     <visual>
-      <origin xyz="0 0 0" rpy="0 0 0"/>
-      <geometry>
-        <mesh filename="package://g1_description/meshes/head_link.STL"/>
-      </geometry>
-      <material name="">
-        <color rgba="0.2 0.2 0.2 1"/>
-      </material>
-    </visual>
-    <collision>
-      <origin xyz="0.055 0.055 0.48" rpy="0 0 0"/>
-      <geometry>
-      <sphere radius="0.01"/>
-      </geometry>
-    </collision>
-    <collision>
-      <origin xyz="0.055 -0.055 0.48" rpy="0 0 0"/>
-      <geometry>
-      <sphere radius="0.01"/>
-      </geometry>
-    </collision>
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