Commit message: Made fixes to the joint_state_controller and camera position

File: robots/g1_description/xacro/gazebo.xacro (robot description, xacro)
@@ -27,5 +27,5 @@
     </sensor>
   </gazebo>
-  <gazebo reference="base">
+  <gazebo reference="pelvis_contour_link">
     <turnGravityOff>false</turnGravityOff>
   </gazebo>
@@ -38,4 +38,5 @@
   <gazebo reference="head_link">
     <sensor type="camera" name="realsense_rgb_camera">
+      <pose>0.06 0 0 0 0 0</pose>  <!-- Añade esta línea -->
       <update_rate>30.0</update_rate>
       <camera>
@@ -67,4 +68,5 @@
     </sensor>
     <sensor type="depth" name="realsense_depth_camera">
+      <pose>0.06 0 0 0 0 0</pose>  <!-- Añade esta línea -->
       <update_rate>30.0</update_rate>
       <camera>

File: robots/g1_description/xacro/robot.xacro (robot description, xacro)
@@ -248,5 +248,5 @@
   <link name="realsense_rgb_frame" />
   <joint name="realsense_rgb_joint" type="fixed">
-    <origin xyz="0.06 0 0.48" rpy="0 0 0" />
+    <origin xyz="0.06 0 0.48" rpy="-1.57079632679 0 -1.57079632679" />
     <parent link="head_link" />
     <child link="realsense_rgb_frame" />
@@ -254,5 +254,5 @@
   <link name="realsense_depth_frame" />
   <joint name="realsense_depth_joint" type="fixed">
-    <origin xyz="0.06 0 0.48" rpy="0 0 0" />
+    <origin xyz="0.06 0 0.48" rpy="-1.57079632679 0 -1.57079632679" />
     <parent link="head_link" />
     <child link="realsense_depth_frame" />

Commit message: modified camera angle

File: robots/g1_description/xacro/gazebo.xacro (robot description, xacro)
@@ -37,5 +37,5 @@
   <gazebo reference="head_link">
     <sensor type="camera" name="realsense_rgb_camera">
-      <pose>0.06 0 0 0 0 0</pose>
+      <pose>0.06 0 0 0 0.436 0</pose>
       <update_rate>30.0</update_rate>
       <camera>
@@ -67,5 +67,5 @@
     </sensor>
     <sensor type="depth" name="realsense_depth_camera">
-      <pose>0.06 0 0 0 0 0</pose>
+      <pose>0.06 0 0 0 0.436 0</pose>
       <update_rate>30.0</update_rate>
       <camera>

File: robots/g1_description/xacro/robot.xacro (robot description, xacro)
@@ -248,5 +248,5 @@
   <link name="realsense_rgb_frame" />
   <joint name="realsense_rgb_joint" type="fixed">
-    <origin xyz="0.06 0 0.48" rpy="-1.57079632679 0 -1.57079632679" />
+    <origin xyz="0.06 0 0.48" rpy="-2.006 0 -1.57079632679" />
     <parent link="head_link" />
     <child link="realsense_rgb_frame" />
@@ -254,5 +254,5 @@
   <link name="realsense_depth_frame" />
   <joint name="realsense_depth_joint" type="fixed">
-    <origin xyz="0.06 0 0.48" rpy="-1.57079632679 0 -1.57079632679" />
+    <origin xyz="0.06 0 0.48" rpy="-2.006 0 -1.57079632679" />
     <parent link="head_link" />
     <child link="realsense_depth_frame" />
@@ -261,5 +261,5 @@
   <link name="camera_link">
     <visual>
-      <origin xyz="0 0 0" rpy="0 0 0" />
+      <origin xyz="0 0 0" rpy="0 0.436 0" />
       <geometry>
         <box size="0.01 0.01 0.01" />
@@ -272,5 +272,5 @@
   <!-- Camera joint - posicionada en la parte frontal de la cabeza -->
   <joint name="camera_joint" type="fixed">
-    <origin xyz="0.06 0 0.48" rpy="0 0 0" />
+    <origin xyz="0.06 0 0.48" rpy="0 0.436 0" />
     <parent link="head_link" />
     <child link="camera_link" />
@@ -279,5 +279,5 @@
   <link name="camera_optical_frame" />
   <joint name="camera_optical_joint" type="fixed">
-    <origin xyz="0 0 0" rpy="-1.57079632679 0 -1.57079632679" />
+    <origin xyz="0 0 0" rpy="-1.57079632679 0.436 -1.57079632679" />
     <parent link="camera_link" />
     <child link="camera_optical_frame" />
